Commit message: repaired the urdf, getting there

File: catkin_ws/src/sailrobot/urdf/sailboat.urdf (robot description, URDF)
Before this commit: robot sailboat, 3 links, 0 joints
Links:
- added link base_rudder
- added link base_sail
- added link world
Joints:
- added joint hull_rudder: type fixed, parent base_hull, child base_rudder, origin xyz=0 -0.1 0
- added joint hull_sail: type fixed, parent base_hull, child base_sail, origin xyz=0 0.05 0
- added joint rudder_angle: type revolute, parent base_rudder, child sailboat_rudder, origin xyz=0 0 -0.03, axis 0 0 1, limit lower=-0.78 upper=0.78 effort=100 velocity=1
- added joint sail_angle: type revolute, parent base_sail, child sailboat_sail, origin xyz=0 0 1, axis 0 0 1, limit lower=-1.57 upper=1.57 effort=100 velocity=1
- added joint world_hull: type floating, parent world, child base_hull

Commit message: working urdf

File: catkin_ws/src/sailrobot/urdf/sailboat.urdf (robot description, URDF)
Before this commit: robot sailboat, 6 links, 5 joints
Links:
- added link base_hull_Y
- added link base_hull_Z
- link base_hull: geometry visual cylinder length=2.0 radius=0.1
Joints:
- removed joint world_hull
- added joint world_hull_X: type continuous, parent base_hull_Y, child base_hull, axis 1 0 0
- added joint world_hull_Y: type continuous, parent base_hull_Z, child base_hull_Y, axis 0 1 0
- added joint world_hull_Z: type continuous, parent world, child base_hull_Z, axis 0 0 1

Commit message: working transform broadcaster with corresponding launch for rviz and mapviz

File: catkin_ws/src/sailrobot/urdf/sailboat.urdf (robot description, URDF)
Before this commit: robot sailboat, 8 links, 7 joints
Links:
- removed link base_hull_Y
- removed link base_hull_Z
- link sailboat_rudder: geometry visual box size=0.01 0.1 0.2
- link sailboat_sail: geometry visual box size=0.01 0.5 1
Joints:
- removed joint world_hull_X
- removed joint world_hull_Y
- removed joint world_hull_Z
- added joint world_hull: type floating, parent world, child base_hull
- joint hull_rudder: origin xyz=0 -0.1 0 -> xyz=0 -0.4 0
- joint rudder_angle: origin xyz=0 0 -0.03 -> xyz=0 0 -0.1
- joint sail_angle: origin xyz=0 0 1 -> xyz=0 0 0.5
